Commit message: * Fixed wrist bracket z offset

File: urdf/x_demo.urdf (robot description, URDF)
Before this commit: robot arm_demo, 9 links, 8 joints
Joints:
- joint shoulder_bracket/OUTPUT_INTERFACE: origin xyz=0 .04235 .05715 rpy=-1.57075 0 0 -> xyz=0 .04235 .04015 rpy=-1.57075 0 0

File: urdf/x_wrist_bracket.xacro (robot description, xacro)
@@ -26,6 +26,6 @@
     <parent link="${name}/INPUT_INTERFACE"/>
     <child link="${child}/INPUT_INTERFACE"/>
-<!--    <origin xyz="0 .03685 .05715" rpy="-1.57075 0 3.14157"/>-->
-    <origin xyz="0 .04235 .05715" rpy="-1.57075 0 0"/>
+<!--    <origin xyz="0 .03685 .05715" rpy="-1.57075 0 3.14157"/> -->
+    <origin xyz="0 .04235 .04015" rpy="-1.57075 0 0"/>
   </joint>
   <gazebo reference="${name}/INPUT_INTERFACE">
