Commit message: Removed comment

File: urdf/x_wrist_bracket.xacro (robot description, xacro)
@@ -26,5 +26,4 @@
     <parent link="${name}/INPUT_INTERFACE"/>
     <child link="${child}/INPUT_INTERFACE"/>
-<!--    <origin xyz="0 .03685 .05715" rpy="-1.57075 0 3.14157"/> -->
     <origin xyz="0 .04235 .04015" rpy="-1.57075 0 0"/>
   </joint>
