Commit message: Update plugin controller structure

File: hebiros_description/urdf/1_dof.xacro (robot description, xacro)
@@ -43,10 +43,6 @@
   </joint>
   <!-- joints -->
-  <xacro:x5 joint="HEBI/base" child="shoulder_bracket"/>
-  <xacro:x_wrist_bracket name="shoulder_bracket" child="HEBI/shoulder"/>
-  <xacro:x5 joint="HEBI/shoulder" child="shoulder_elbow"/>
-  <xacro:x_tube_link name="shoulder_elbow" child="HEBI/elbow" length="0.33" twist="0"/>
-  <xacro:x5 joint="HEBI/elbow" child="elbow_end"/>
-  <xacro:x_tube_link name="elbow_end" child="end_effector" length="0.325" twist="0"/>
+  <xacro:x5 joint="HEBI/base" child="base_end"/>
+  <xacro:x_tube_link name="base_end" child="end_effector" length="0.33" twist="0"/>
   <!-- end link -->
   <link name="end_effector/INPUT_INTERFACE">

File: hebiros_description/urdf/x5.xacro (robot description, xacro)
@@ -29,5 +29,5 @@
       <axis xyz="0 0 1"/>
       <limit effort="9.0" lower="-10.0" upper="10.0" velocity="2.208932"/>
-      <dynamics damping="0.2" friction="0.2"/>
+      <dynamics damping="0.5" friction="0.5"/>
     </joint>
     <transmission name="${joint}/transmission">
