Commit message: Added switching x models via urdf

File: hebiros_description/urdf/1_dof.urdf (robot description, URDF)
Before this commit: robot arm_demo, 5 links, 4 joints
Joints:
- removed joint HEBI/base
- added joint HEBI/base/X5-4: type revolute, parent HEBI/base/INPUT_INTERFACE, child base_end/INPUT_INTERFACE, origin xyz=0 0 0.031 rpy=0 0 0, axis 0 0 1, limit lower=-10.0 upper=10.0 effort=9.0 velocity=2.208932

File: hebiros_description/urdf/1_dof.xacro (robot description, xacro)
@@ -43,5 +43,5 @@
   </joint>
   <!-- joints -->
-  <xacro:x5 joint="HEBI/base" child="base_end"/>
+  <xacro:x5 joint="HEBI/base" child="base_end" model="X5-4"/>
   <xacro:x_tube_link name="base_end" child="end_effector" length="0.33" twist="0"/>
   <!-- end link -->

File: hebiros_description/urdf/x5.xacro (robot description, xacro)
@@ -2,5 +2,6 @@
 <robot xmlns:xacro="http://www.ros.org/wiki/xacro">
   <!-- NOTE: joint must match the name of the module -->
-  <xacro:macro name="x5" params="joint child">
+  <xacro:macro name="x5" params="joint child model">
+  <xacro:property name="model_name" value="${model}"/>
     <link name="${joint}/INPUT_INTERFACE">
       <visual>
@@ -23,12 +24,34 @@
       </inertial>
     </link>
-    <joint name="${joint}" type="revolute">
-      <parent link="${joint}/INPUT_INTERFACE"/>
-      <child link="${child}/INPUT_INTERFACE"/>
-      <origin xyz="0 0 0.031" rpy="0 0 0"/>
-      <axis xyz="0 0 1"/>
-      <limit effort="9.0" lower="-10.0" upper="10.0" velocity="2.208932"/>
-      <dynamics damping="0.5" friction="0.5"/>
-    </joint>
+    <xacro:if value="${model_name == 'X5-1'}">
+      <joint name="${joint}/X5-1" type="revolute">
+        <parent link="${joint}/INPUT_INTERFACE"/>
+        <child link="${child}/INPUT_INTERFACE"/>
+        <origin xyz="0 0 0.031" rpy="0 0 0"/>
+        <axis xyz="0 0 1"/>
+        <limit effort="9.0" lower="-10.0" upper="10.0" velocity="2.208932"/>
+        <dynamics damping="0.5" friction="0.5"/>
+      </joint>
+    </xacro:if>
+    <xacro:if value="${model_name == 'X5-4'}">
+      <joint name="${joint}/X5-4" type="revolute">
+        <parent link="${joint}/INPUT_INTERFACE"/>
+        <child link="${child}/INPUT_INTERFACE"/>
+        <origin xyz="0 0 0.031" rpy="0 0 0"/>
+        <axis xyz="0 0 1"/>
+        <limit effort="9.0" lower="-10.0" upper="10.0" velocity="2.208932"/>
+        <dynamics damping="0.5" friction="0.5"/>
+      </joint>
+    </xacro:if>
+    <xacro:if value="${model_name == 'X5-9'}">
+      <joint name="${joint}/X5-9" type="revolute">
+        <parent link="${joint}/INPUT_INTERFACE"/>
+        <child link="${child}/INPUT_INTERFACE"/>
+        <origin xyz="0 0 0.031" rpy="0 0 0"/>
+        <axis xyz="0 0 1"/>
+        <limit effort="9.0" lower="-10.0" upper="10.0" velocity="2.208932"/>
+        <dynamics damping="0.5" friction="0.5"/>
+      </joint>
+    </xacro:if>
     <transmission name="${joint}/transmission">
     <type>transmission_interface/SimpleTransmission</type>

File: hebiros_description/urdf/x_demo.urdf (robot description, URDF)
Before this commit: robot arm_demo, 9 links, 8 joints
Joints:
- removed joint HEBI/base
- removed joint HEBI/elbow
- removed joint HEBI/shoulder
- added joint HEBI/base/X5-1: type revolute, parent HEBI/base/INPUT_INTERFACE, child shoulder_bracket/INPUT_INTERFACE, origin xyz=0 0 0.031 rpy=0 0 0, axis 0 0 1, limit lower=-10.0 upper=10.0 effort=9.0 velocity=2.208932
- added joint HEBI/elbow/X5-9: type revolute, parent HEBI/elbow/INPUT_INTERFACE, child elbow_end/INPUT_INTERFACE, origin xyz=0 0 0.031 rpy=0 0 0, axis 0 0 1, limit lower=-10.0 upper=10.0 effort=9.0 velocity=2.208932
- added joint HEBI/shoulder/X5-4: type revolute, parent HEBI/shoulder/INPUT_INTERFACE, child shoulder_elbow/INPUT_INTERFACE, origin xyz=0 0 0.031 rpy=0 0 0, axis 0 0 1, limit lower=-10.0 upper=10.0 effort=9.0 velocity=2.208932

File: hebiros_description/urdf/x_demo.xacro (robot description, xacro)
@@ -43,9 +43,9 @@
   </joint>
   <!-- joints -->
-  <xacro:x5 joint="HEBI/base" child="shoulder_bracket"/>
+  <xacro:x5 joint="HEBI/base" child="shoulder_bracket" model="X5-1"/>
   <xacro:x_wrist_bracket name="shoulder_bracket" child="HEBI/shoulder"/>
-  <xacro:x5 joint="HEBI/shoulder" child="shoulder_elbow"/>
+  <xacro:x5 joint="HEBI/shoulder" child="shoulder_elbow" model="X5-4"/>
   <xacro:x_tube_link name="shoulder_elbow" child="HEBI/elbow" length="0.33" twist="0"/>
-  <xacro:x5 joint="HEBI/elbow" child="elbow_end"/>
+  <xacro:x5 joint="HEBI/elbow" child="elbow_end" model="X5-9"/>
   <xacro:x_tube_link name="elbow_end" child="end_effector" length="0.325" twist="0"/>
   <!-- end link -->

Commit message: Added setting command lifetime and changed symbol for x models to hyphen

File: hebiros_description/urdf/1_dof.urdf (robot description, URDF)
Before this commit: robot arm_demo, 5 links, 4 joints
Joints:
- removed joint HEBI/base/X5-4

File: hebiros_description/urdf/x5.xacro (robot description, xacro)
@@ -24,6 +24,6 @@
       </inertial>
     </link>
-    <xacro:if value="${model_name == 'X5-1'}">
-      <joint name="${joint}/X5-1" type="revolute">
+    <xacro:if value="${model_name == 'X5_1'}">
+      <joint name="${joint}/X5_1" type="revolute">
         <parent link="${joint}/INPUT_INTERFACE"/>
         <child link="${child}/INPUT_INTERFACE"/>
@@ -34,6 +34,6 @@
       </joint>
     </xacro:if>
-    <xacro:if value="${model_name == 'X5-4'}">
-      <joint name="${joint}/X5-4" type="revolute">
+    <xacro:if value="${model_name == 'X5_4'}">
+      <joint name="${joint}/X5_4" type="revolute">
         <parent link="${joint}/INPUT_INTERFACE"/>
         <child link="${child}/INPUT_INTERFACE"/>
@@ -44,6 +44,6 @@
       </joint>
     </xacro:if>
-    <xacro:if value="${model_name == 'X5-9'}">
-      <joint name="${joint}/X5-9" type="revolute">
+    <xacro:if value="${model_name == 'X5_9'}">
+      <joint name="${joint}/X5_9" type="revolute">
         <parent link="${joint}/INPUT_INTERFACE"/>
         <child link="${child}/INPUT_INTERFACE"/>

File: hebiros_description/urdf/x_demo.urdf (robot description, URDF)
Before this commit: robot arm_demo, 9 links, 8 joints
Joints:
- removed joint HEBI/base/X5-4
- removed joint HEBI/elbow/X5-4
- removed joint HEBI/shoulder/X5-4
- added joint HEBI/base/X5_4: type revolute, parent HEBI/base/INPUT_INTERFACE, child shoulder_bracket/INPUT_INTERFACE, origin xyz=0 0 0.031 rpy=0 0 0, axis 0 0 1, limit lower=-10.0 upper=10.0 effort=90.0 velocity=2.208932
- added joint HEBI/elbow/X5_4: type revolute, parent HEBI/elbow/INPUT_INTERFACE, child elbow_end/INPUT_INTERFACE, origin xyz=0 0 0.031 rpy=0 0 0, axis 0 0 1, limit lower=-10.0 upper=10.0 effort=90.0 velocity=2.208932
- added joint HEBI/shoulder/X5_4: type revolute, parent HEBI/shoulder/INPUT_INTERFACE, child shoulder_elbow/INPUT_INTERFACE, origin xyz=0 0 0.031 rpy=0 0 0, axis 0 0 1, limit lower=-10.0 upper=10.0 effort=90.0 velocity=2.208932

File: hebiros_description/urdf/x_demo.xacro (robot description, xacro)
@@ -43,9 +43,9 @@
   </joint>
   <!-- joints -->
-  <xacro:x5 joint="HEBI/base" child="shoulder_bracket" model="X5-4"/>
+  <xacro:x5 joint="HEBI/base" child="shoulder_bracket" model="X5_4"/>
   <xacro:x_wrist_bracket name="shoulder_bracket" child="HEBI/shoulder"/>
-  <xacro:x5 joint="HEBI/shoulder" child="shoulder_elbow" model="X5-4"/>
+  <xacro:x5 joint="HEBI/shoulder" child="shoulder_elbow" model="X5_4"/>
   <xacro:x_tube_link name="shoulder_elbow" child="HEBI/elbow" length="0.33" twist="0"/>
-  <xacro:x5 joint="HEBI/elbow" child="elbow_end" model="X5-4"/>
+  <xacro:x5 joint="HEBI/elbow" child="elbow_end" model="X5_4"/>
   <xacro:x_tube_link name="elbow_end" child="end_effector" length="0.325" twist="0"/>
   <!-- end link -->

Commit message: Fix effort control

File: hebiros_description/urdf/1_dof.urdf (robot description, URDF)
Before this commit: robot arm_demo, 5 links, 3 joints
Links:
- link base_end/INPUT_INTERFACE: geometry collision cylinder length=0.33 radius=.015875; collision mesh filename=package://hebiros_description/meshes/x_mounting_bracket.stl

File: hebiros_description/urdf/x5.xacro (robot description, xacro)
@@ -30,6 +30,6 @@
         <origin xyz="0 0 0.031" rpy="0 0 0"/>
         <axis xyz="0 0 1"/>
-        <limit effort="90.0" lower="-10.0" upper="10.0" velocity="2.208932"/>
-        <dynamics damping="0.2" friction="0.2"/>
+        <limit effort="9.0" lower="-10.0" upper="10.0" velocity="2.208932"/>
+        <dynamics damping="0.5" friction="0.5"/>
       </joint>
     </xacro:if>
@@ -40,6 +40,6 @@
         <origin xyz="0 0 0.031" rpy="0 0 0"/>
         <axis xyz="0 0 1"/>
-        <limit effort="90.0" lower="-10.0" upper="10.0" velocity="2.208932"/>
-        <dynamics damping="0.2" friction="0.2"/>
+        <limit effort="9.0" lower="-10.0" upper="10.0" velocity="2.208932"/>
+        <dynamics damping="0.5" friction="0.5"/>
       </joint>
     </xacro:if>
@@ -50,6 +50,6 @@
         <origin xyz="0 0 0.031" rpy="0 0 0"/>
         <axis xyz="0 0 1"/>
-        <limit effort="90.0" lower="-10.0" upper="10.0" velocity="2.208932"/>
-        <dynamics damping="0.2" friction="0.2"/>
+        <limit effort="9.0" lower="-10.0" upper="10.0" velocity="2.208932"/>
+        <dynamics damping="0.5" friction="0.5"/>
       </joint>
     </xacro:if>

File: hebiros_description/urdf/x_demo.urdf (robot description, URDF)
Before this commit: robot arm_demo, 9 links, 8 joints
Links:
- link elbow_end/INPUT_INTERFACE: geometry collision cylinder length=0.325 radius=.015875; collision mesh filename=package://hebiros_description/meshes/x_mounting_bracket.stl
- link shoulder_elbow/INPUT_INTERFACE: geometry collision cylinder length=0.33 radius=.015875; collision mesh filename=package://hebiros_description/meshes/x_mounting_bracket.stl
Joints:
- joint HEBI/base/X5_4: limit lower=-10.0 upper=10.0 effort=90.0 velocity=2.208932 -> lower=-10.0 upper=10.0 effort=9.0 velocity=2.208932
- joint HEBI/elbow/X5_4: limit lower=-10.0 upper=10.0 effort=90.0 velocity=2.208932 -> lower=-10.0 upper=10.0 effort=9.0 velocity=2.208932
- joint HEBI/shoulder/X5_4: limit lower=-10.0 upper=10.0 effort=90.0 velocity=2.208932 -> lower=-10.0 upper=10.0 effort=9.0 velocity=2.208932

File: hebiros_description/urdf/x_demo.xacro (robot description, xacro)
@@ -46,7 +46,7 @@
   <xacro:x_wrist_bracket name="shoulder_bracket" child="HEBI/shoulder"/>
   <xacro:x5 joint="HEBI/shoulder" child="shoulder_elbow" model="X5_4"/>
-  <xacro:x_tube_link name="shoulder_elbow" child="HEBI/elbow" length="0.33" twist="0"/>
+  <xacro:x_tube_link name="shoulder_elbow" child="HEBI/elbow" length="0.33" twist="0.7"/>
   <xacro:x5 joint="HEBI/elbow" child="elbow_end" model="X5_4"/>
-  <xacro:x_tube_link name="elbow_end" child="end_effector" length="0.325" twist="0"/>
+  <xacro:x_tube_link name="elbow_end" child="end_effector" length="0.325" twist="0.6"/>
   <!-- end link -->
   <link name="end_effector/INPUT_INTERFACE">
