Commit message: Finished adding light brackets, and making small tweaks to heavy brackets (don't add color to the collision objects!)

File: hebiros_description/urdf/x5_heavy_left_inside_bracket.xacro (robot description, xacro)
@@ -23,5 +23,4 @@
         <mesh filename="package://hebiros_description/meshes/PM-2149-01.stl" scale="0.001 0.001 0.001"/>
       </geometry>
-      <xacro:black_material/>
     </collision>
     <collision>
@@ -30,5 +29,4 @@
         <mesh filename="package://hebiros_description/meshes/PM-2150-01L.stl" scale="0.001 0.001 0.001"/>
       </geometry>
-      <xacro:black_material/>
     </collision>
     <!-- NOTE: inertia is just modelled as small sphere, and could be improved. -->

File: hebiros_description/urdf/x5_heavy_left_outside_bracket.xacro (robot description, xacro)
@@ -23,5 +23,4 @@
         <mesh filename="package://hebiros_description/meshes/PM-2149-01.stl" scale="0.001 0.001 0.001"/>
       </geometry>
-      <xacro:black_material/>
     </collision>
     <collision>
@@ -30,5 +29,4 @@
         <mesh filename="package://hebiros_description/meshes/PM-2150-01L.stl" scale="0.001 0.001 0.001"/>
       </geometry>
-      <xacro:black_material/>
     </collision>
     <!-- NOTE: inertia is just modelled as small sphere, and could be improved. -->

File: hebiros_description/urdf/x5_heavy_right_inside_bracket.xacro (robot description, xacro)
@@ -23,5 +23,4 @@
         <mesh filename="package://hebiros_description/meshes/PM-2149-01.stl" scale="0.001 0.001 0.001"/>
       </geometry>
-      <xacro:black_material/>
     </collision>
     <collision>
@@ -30,5 +29,4 @@
         <mesh filename="package://hebiros_description/meshes/PM-2150-01R.stl" scale="0.001 0.001 0.001"/>
       </geometry>
-      <xacro:black_material/>
     </collision>
     <!-- NOTE: inertia is just modelled as small sphere, and could be improved. -->

File: hebiros_description/urdf/x5_heavy_right_outside_bracket.xacro (robot description, xacro)
@@ -23,5 +23,4 @@
         <mesh filename="package://hebiros_description/meshes/PM-2149-01.stl" scale="0.001 0.001 0.001"/>
       </geometry>
-      <xacro:black_material/>
     </collision>
     <collision>
@@ -30,5 +29,4 @@
         <mesh filename="package://hebiros_description/meshes/PM-2150-01R.stl" scale="0.001 0.001 0.001"/>
       </geometry>
-      <xacro:black_material/>
     </collision>
     <!-- NOTE: inertia is just modelled as small sphere, and could be improved. -->

File: hebiros_description/urdf/x_library.xacro (robot description, xacro)
@@ -5,4 +5,6 @@
   <xacro:include filename="./x5.xacro"/>
   <xacro:include filename="./x8.xacro"/>
+  <xacro:include filename="./x5_light_left_bracket.xacro"/>
+  <xacro:include filename="./x5_light_right_bracket.xacro"/>
   <xacro:include filename="./x5_heavy_left_outside_bracket.xacro"/>
   <xacro:include filename="./x5_heavy_left_inside_bracket.xacro"/>

File: hebiros_description/urdf/x_series_common.xacro (robot description, xacro)
@@ -17,3 +17,8 @@
     </material>
   </xacro:macro>
+  <xacro:macro name="beige_material">
+    <material name="beige">
+      <color rgba="0.96 0.945 0.871 1"/>
+    </material>
+  </xacro:macro>
 </robot>
