Commit message: - Updated heavy brackets to match HEBI standard part library. - Created a "library" so you only need to include one xacro file.

File: hebiros_description/urdf/x_demo.urdf (robot description, URDF)
Before this commit: robot arm_demo, 9 links, 8 joints
Links:
- link shoulder_bracket/INPUT_INTERFACE: mass 0.1 -> 0.215; geometry collision mesh filename=package://hebiros_description/meshes/PM-2149-01.stl scale=0.001 0.001 0.001; collision mesh filename=package://hebiros_description/meshes/PM-2150-01R.stl scale=0.001 0.001 0.001
Joints:
- joint elbow_end/OUTPUT_JOINT: origin xyz=0.325 -0.0189260017537 0.0135342086627 rpy=1.9 0 0 -> xyz=0.325 -2.44929359829e-18 0.0 rpy=3.14159265359 0 0
- joint shoulder_bracket/OUTPUT_INTERFACE: origin xyz=0 .04235 .04015 rpy=-1.57075 0 0 -> xyz=0 .0225 .055 rpy=1.57079632679 0 0
- joint shoulder_elbow/OUTPUT_JOINT: origin xyz=0.33 -0.00494807918509 0.0393782484342 rpy=0.25 0 0 -> xyz=0.33 -2.44929359829e-18 0.0 rpy=3.14159265359 0 0

File: hebiros_description/urdf/x_demo.xacro (robot description, xacro)
@@ -2,12 +2,5 @@
 <robot xmlns:xacro="http://www.ros.org/wiki/xacro" name="arm_demo">
   <!-- *************************** XACRO MACROS *************************** -->
-  <xacro:property name="PI" value="3.1415926535897931" />
-  <!-- load macros for modules -->
-  <xacro:include filename="./x_series_common.xacro"/>
-  <xacro:include filename="./x5.xacro"/>
-  <xacro:include filename="./x8.xacro"/>
-  <xacro:include filename="./x_shoulder_bracket.xacro"/>
-  <xacro:include filename="./x_wrist_bracket.xacro"/>
-  <xacro:include filename="./x_tube_link.xacro"/>
+  <xacro:include filename="./x_library.xacro"/>
   <!-- ************************* ROBOT DEFINITION ************************* -->
   <link name="world" />
@@ -45,9 +38,9 @@
   <!-- joints -->
   <xacro:x5 joint="HEBI/base" child="shoulder_bracket" model="X5_4"/>
-  <xacro:x_wrist_bracket name="shoulder_bracket" child="HEBI/shoulder"/>
+  <xacro:x5_heavy_right_inside_bracket name="shoulder_bracket" child="HEBI/shoulder"/>
   <xacro:x5 joint="HEBI/shoulder" child="shoulder_elbow" model="X5_4"/>
-  <xacro:x_tube_link name="shoulder_elbow" child="HEBI/elbow" extension="0.33" twist="0.25"/>
+  <xacro:x_tube_link name="shoulder_elbow" child="HEBI/elbow" extension="0.33" twist="${PI}"/>
   <xacro:x5 joint="HEBI/elbow" child="elbow_end" model="X5_4"/>
-  <xacro:x_tube_link name="elbow_end" child="end_effector" extension="0.325" twist="1.9"/>
+  <xacro:x_tube_link name="elbow_end" child="end_effector" extension="0.325" twist="${PI}"/>
   <!-- end link -->
   <link name="end_effector/INPUT_INTERFACE">

Commit message: Change the meshes for the tube brackets to include caps (reference the complete assembly)

File: hebiros_description/urdf/x_demo.urdf (robot description, URDF)
Before this commit: robot arm_demo, 9 links, 8 joints
Links:
- link elbow_end/INPUT_INTERFACE: geometry collision cylinder length=0.2996 radius=.016; collision mesh filename=package://hebiros_description/meshes/A-2038-02.stl
- link shoulder_elbow/INPUT_INTERFACE: geometry collision cylinder length=0.3046 radius=.016; collision mesh filename=package://hebiros_description/meshes/A-2038-02.stl

File: hebiros_description/urdf/x_tube_link.xacro (robot description, xacro)
@@ -9,5 +9,5 @@
         <origin xyz="0 0 0" rpy="0 0 0" />
         <geometry>
-          <mesh filename="package://hebiros_description/meshes/PM-2146-02.stl" scale=".001 .001 .001"/>
+          <mesh filename="package://hebiros_description/meshes/A-2038-02.stl"/>
         </geometry>
         <xacro:black_material/>
@@ -21,7 +21,7 @@
       </visual>
       <visual>
-        <origin xyz="${extension} ${sin(-twist) * edge_to_center} ${edge_to_center * (1 + cos(-twist))}" rpy="${-twist + 3.1415} 0 3.1415"/>
+        <origin xyz="${extension} ${sin(-twist) * edge_to_center} ${edge_to_center * (1 + cos(-twist))}" rpy="${-twist} 0 0"/>
         <geometry>
-          <mesh filename="package://hebiros_description/meshes/PM-2147-02.stl" scale=".001 .001 .001"/>
+          <mesh filename="package://hebiros_description/meshes/A-2039-02.stl"/>
         </geometry>
         <xacro:black_material/>
@@ -30,5 +30,5 @@
         <origin xyz="0 0 0" rpy="0 0 0" />
         <geometry>
-          <mesh filename="package://hebiros_description/meshes/PM-2146-02.stl" scale=".001 .001 .001"/>
+          <mesh filename="package://hebiros_description/meshes/A-2038-02.stl"/>
         </geometry>
       </collision>
@@ -40,7 +40,7 @@
       </collision>
       <collision>
-        <origin xyz="${extension} ${sin(-twist) * edge_to_center} ${edge_to_center * (1 + cos(-twist))}" rpy="${-twist + 3.1415} 0 3.1415"/>
+        <origin xyz="${extension} ${sin(-twist) * edge_to_center} ${edge_to_center * (1 + cos(-twist))}" rpy="${-twist} 0 0"/>
         <geometry>
-          <mesh filename="package://hebiros_description/meshes/PM-2147-02.stl" scale=".001 .001 .001"/>
+          <mesh filename="package://hebiros_description/meshes/A-2039-02.stl"/>
         </geometry>
       </collision>
