Commit message: Update the X5 xacro (adding proper limits, etc) and add the X8.

File: hebiros_description/urdf/x8.xacro (robot description, xacro)
@@ -2,5 +2,5 @@
 <robot xmlns:xacro="http://www.ros.org/wiki/xacro">
   <!-- NOTE: joint must match the name of the module -->
-  <xacro:macro name="x5" params="joint child model">
+  <xacro:macro name="x8" params="joint child model">
   <xacro:property name="model_name" value="${model}"/>
     <link name="${joint}/INPUT_INTERFACE">
@@ -8,5 +8,5 @@
         <origin xyz="0 0 0" rpy="0 0 3.1415" />
         <geometry>
-          <mesh filename="package://hebiros_description/meshes/x5.stl" scale="0.001 0.001 0.001"/>
+          <mesh filename="package://hebiros_description/meshes/x8.stl" scale="0.001 0.001 0.001"/>
         </geometry>
         <xacro:red_material/>
@@ -15,48 +15,48 @@
         <origin xyz="0 0 0" rpy="0 0 3.1415" />
         <geometry>
-          <mesh filename="package://hebiros_description/meshes/x5.stl" scale="0.001 0.001 0.001"/>
+          <mesh filename="package://hebiros_description/meshes/x8.stl" scale="0.001 0.001 0.001"/>
         </geometry>
       </collision>
       <inertial>
-        <origin xyz="-0.0142 -0.0031 0.0165" rpy="0 0 0" />
-        <xacro:if value="${model_name == 'X5_1'}">
-          <mass value="0.315"/>
+        <origin xyz="-0.0145 -0.0031 0.0242" rpy="0 0 0" />
+        <xacro:if value="${model_name == 'X8_3'}">
+          <mass value="0.460"/>
         </xacro:if>
-        <xacro:if value="${model_name == 'X5_4'}">
-          <mass value="0.335"/>
+        <xacro:if value="${model_name == 'X8_9'}">
+          <mass value="0.480"/>
         </xacro:if>
-        <xacro:if value="${model_name == 'X5_9'}">
-          <mass value="0.360"/>
+        <xacro:if value="${model_name == 'X8_16'}">
+          <mass value="0.500"/>
         </xacro:if>
-        <inertia ixx="0.00015" iyy="0.000255" izz="0.000350" ixy="0.0000341" ixz="0.0000118" iyz="0.00000229"/>
+        <inertia ixx="0.000246" iyy="0.000380" izz="0.000463" ixy="0.0000444" ixz="0.0000266" iyz="0.00000422"/>
       </inertial>
     </link>
-    <xacro:if value="${model_name == 'X5_1'}">
-      <joint name="${joint}/X5_1" type="continuous">
+    <xacro:if value="${model_name == 'X8_3'}">
+      <joint name="${joint}/X8_3" type="continuous">
         <parent link="${joint}/INPUT_INTERFACE"/>
         <child link="${child}/INPUT_INTERFACE"/>
-        <origin xyz="0 0 0.031" rpy="0 0 0"/>
+        <origin xyz="0 0 0.045" rpy="0 0 0"/>
         <axis xyz="0 0 1"/>
-        <limit effort="2.5" velocity="90"/>
+        <limit effort="7" velocity="84"/>
         <dynamics damping="0.5" friction="0.5"/>
       </joint>
     </xacro:if>
-    <xacro:if value="${model_name == 'X5_4'}">
-      <joint name="${joint}/X5_4" type="continuous">
+    <xacro:if value="${model_name == 'X8_9'}">
+      <joint name="${joint}/X8_9" type="continuous">
         <parent link="${joint}/INPUT_INTERFACE"/>
         <child link="${child}/INPUT_INTERFACE"/>
-        <origin xyz="0 0 0.031" rpy="0 0 0"/>
+        <origin xyz="0 0 0.045" rpy="0 0 0"/>
         <axis xyz="0 0 1"/>
-        <limit effort="7.0" velocity="32"/>
+        <limit effort="20" velocity="30"/>
         <dynamics damping="0.5" friction="0.5"/>
       </joint>
     </xacro:if>
-    <xacro:if value="${model_name == 'X5_9'}">
-      <joint name="${joint}/X5_9" type="continuous">
+    <xacro:if value="${model_name == 'X8_16'}">
+      <joint name="${joint}/X8_16" type="continuous">
         <parent link="${joint}/INPUT_INTERFACE"/>
         <child link="${child}/INPUT_INTERFACE"/>
-        <origin xyz="0 0 0.031" rpy="0 0 0"/>
+        <origin xyz="0 0 0.045" rpy="0 0 0"/>
         <axis xyz="0 0 1"/>
-        <limit effort="13.0" velocity="14"/>
+        <limit effort="38" velocity="15"/>
         <dynamics damping="0.5" friction="0.5"/>
       </joint>

File: hebiros_description/urdf/x_demo.urdf (robot description, URDF)
Before this commit: robot arm_demo, 9 links, 8 joints
Links:
- link HEBI/base/INPUT_INTERFACE: geometry collision mesh filename=package://hebiros_description/meshes/x5.stl scale=0.001 0.001 0.001; visual mesh filename=package://hebiros_description/meshes/x5.stl scale=0.001 0.001 0.001
- link HEBI/elbow/INPUT_INTERFACE: geometry collision mesh filename=package://hebiros_description/meshes/x5.stl scale=0.001 0.001 0.001; visual mesh filename=package://hebiros_description/meshes/x5.stl scale=0.001 0.001 0.001
- link HEBI/shoulder/INPUT_INTERFACE: geometry collision mesh filename=package://hebiros_description/meshes/x5.stl scale=0.001 0.001 0.001; visual mesh filename=package://hebiros_description/meshes/x5.stl scale=0.001 0.001 0.001
Joints:
- joint HEBI/base/X5_4: limit lower=-10.0 upper=10.0 effort=9.0 velocity=2.208932 -> effort=7.0 velocity=32; type revolute -> continuous
- joint HEBI/elbow/X5_4: limit lower=-10.0 upper=10.0 effort=9.0 velocity=2.208932 -> effort=7.0 velocity=32; type revolute -> continuous
- joint HEBI/shoulder/X5_4: limit lower=-10.0 upper=10.0 effort=9.0 velocity=2.208932 -> effort=7.0 velocity=32; type revolute -> continuous

File: hebiros_description/urdf/x_demo.xacro (robot description, xacro)
@@ -6,4 +6,5 @@
   <xacro:include filename="./x_series_common.xacro"/>
   <xacro:include filename="./x5.xacro"/>
+  <xacro:include filename="./x8.xacro"/>
   <xacro:include filename="./x_shoulder_bracket.xacro"/>
   <xacro:include filename="./x_wrist_bracket.xacro"/>

Commit message: Iamtesch/update urdf (#69)
* Update the X5 xacro (adding proper limits, etc) and add the X8.

* Fixed coordinate system issues with X5 / X8 modules, and updated X tube
link definition to add "twist" parameter and fix dimensions, masses and inertias.

* - Updated heavy brackets to match HEBI standard part library.
- Created a "library" so you only need to include one xacro file.

* Finished adding light brackets, and making small tweaks to heavy
brackets (don't add color to the collision objects!)

* Forgot to remove this line.

* Change the meshes for the tube brackets to include caps (reference the
complete assembly)

File: hebiros_description/urdf/x8.xacro (robot description, xacro)
@@ -2,5 +2,5 @@
 <robot xmlns:xacro="http://www.ros.org/wiki/xacro">
   <!-- NOTE: joint must match the name of the module -->
-  <xacro:macro name="x5" params="joint child model">
+  <xacro:macro name="x8" params="joint child model">
   <xacro:property name="model_name" value="${model}"/>
     <link name="${joint}/INPUT_INTERFACE">
@@ -8,5 +8,5 @@
         <origin xyz="0 0 0" rpy="0 0 0" />
         <geometry>
-          <mesh filename="package://hebiros_description/meshes/x5.stl" scale="0.001 0.001 0.001"/>
+          <mesh filename="package://hebiros_description/meshes/x8.stl" scale="0.001 0.001 0.001"/>
         </geometry>
         <xacro:red_material/>
@@ -15,48 +15,48 @@
         <origin xyz="0 0 0" rpy="0 0 0" />
         <geometry>
-          <mesh filename="package://hebiros_description/meshes/x5.stl" scale="0.001 0.001 0.001"/>
+          <mesh filename="package://hebiros_description/meshes/x8.stl" scale="0.001 0.001 0.001"/>
         </geometry>
       </collision>
       <inertial>
-        <origin xyz="-0.0142 -0.0031 0.0165" rpy="0 0 0" />
-        <xacro:if value="${model_name == 'X5_1'}">
-          <mass value="0.315"/>
+        <origin xyz="-0.0145 -0.0031 0.0242" rpy="0 0 0" />
+        <xacro:if value="${model_name == 'X8_3'}">
+          <mass value="0.460"/>
         </xacro:if>
-        <xacro:if value="${model_name == 'X5_4'}">
-          <mass value="0.335"/>
+        <xacro:if value="${model_name == 'X8_9'}">
+          <mass value="0.480"/>
         </xacro:if>
-        <xacro:if value="${model_name == 'X5_9'}">
-          <mass value="0.360"/>
+        <xacro:if value="${model_name == 'X8_16'}">
+          <mass value="0.500"/>
         </xacro:if>
-        <inertia ixx="0.00015" iyy="0.000255" izz="0.000350" ixy="0.0000341" ixz="0.0000118" iyz="0.00000229"/>
+        <inertia ixx="0.000246" iyy="0.000380" izz="0.000463" ixy="0.0000444" ixz="0.0000266" iyz="0.00000422"/>
       </inertial>
     </link>
-    <xacro:if value="${model_name == 'X5_1'}">
-      <joint name="${joint}/X5_1" type="continuous">
+    <xacro:if value="${model_name == 'X8_3'}">
+      <joint name="${joint}/X8_3" type="continuous">
         <parent link="${joint}/INPUT_INTERFACE"/>
         <child link="${child}/INPUT_INTERFACE"/>
-        <origin xyz="0 0 0.031" rpy="0 0 0"/>
+        <origin xyz="0 0 0.045" rpy="0 0 0"/>
         <axis xyz="0 0 1"/>
-        <limit effort="2.5" velocity="90"/>
+        <limit effort="7" velocity="84"/>
         <dynamics damping="0.5" friction="0.5"/>
       </joint>
     </xacro:if>
-    <xacro:if value="${model_name == 'X5_4'}">
-      <joint name="${joint}/X5_4" type="continuous">
+    <xacro:if value="${model_name == 'X8_9'}">
+      <joint name="${joint}/X8_9" type="continuous">
         <parent link="${joint}/INPUT_INTERFACE"/>
         <child link="${child}/INPUT_INTERFACE"/>
-        <origin xyz="0 0 0.031" rpy="0 0 0"/>
+        <origin xyz="0 0 0.045" rpy="0 0 0"/>
         <axis xyz="0 0 1"/>
-        <limit effort="7.0" velocity="32"/>
+        <limit effort="20" velocity="30"/>
         <dynamics damping="0.5" friction="0.5"/>
       </joint>
     </xacro:if>
-    <xacro:if value="${model_name == 'X5_9'}">
-      <joint name="${joint}/X5_9" type="continuous">
+    <xacro:if value="${model_name == 'X8_16'}">
+      <joint name="${joint}/X8_16" type="continuous">
         <parent link="${joint}/INPUT_INTERFACE"/>
         <child link="${child}/INPUT_INTERFACE"/>
-        <origin xyz="0 0 0.031" rpy="0 0 0"/>
+        <origin xyz="0 0 0.045" rpy="0 0 0"/>
         <axis xyz="0 0 1"/>
-        <limit effort="13.0" velocity="14"/>
+        <limit effort="38" velocity="15"/>
         <dynamics damping="0.5" friction="0.5"/>
       </joint>

File: hebiros_description/urdf/x_demo.urdf (robot description, URDF)
Before this commit: robot arm_demo, 9 links, 8 joints
Links:
- link HEBI/base/INPUT_INTERFACE: geometry collision mesh filename=package://hebiros_description/meshes/x5.stl scale=0.001 0.001 0.001; visual mesh filename=package://hebiros_description/meshes/x5.stl scale=0.001 0.001 0.001
- link HEBI/elbow/INPUT_INTERFACE: geometry collision mesh filename=package://hebiros_description/meshes/x5.stl scale=0.001 0.001 0.001; visual mesh filename=package://hebiros_description/meshes/x5.stl scale=0.001 0.001 0.001
- link HEBI/shoulder/INPUT_INTERFACE: geometry collision mesh filename=package://hebiros_description/meshes/x5.stl scale=0.001 0.001 0.001; visual mesh filename=package://hebiros_description/meshes/x5.stl scale=0.001 0.001 0.001
- link elbow_end/INPUT_INTERFACE: mass 0.01 -> 0.402; geometry collision cylinder length=0.2996 radius=.016; collision mesh filename=package://hebiros_description/meshes/A-2038-02.stl
- link shoulder_bracket/INPUT_INTERFACE: mass 0.1 -> 0.215; geometry collision mesh filename=package://hebiros_description/meshes/PM-2149-01.stl scale=0.001 0.001 0.001; collision mesh filename=package://hebiros_description/meshes/PM-2150-01R.stl scale=0.001 0.001 0.001
- link shoulder_elbow/INPUT_INTERFACE: mass 0.01 -> 0.404; geometry collision cylinder length=0.3046 radius=.016; collision mesh filename=package://hebiros_description/meshes/A-2038-02.stl
Joints:
- joint HEBI/base/X5_4: limit lower=-10.0 upper=10.0 effort=9.0 velocity=2.208932 -> effort=7.0 velocity=32; type revolute -> continuous
- joint HEBI/elbow/X5_4: limit lower=-10.0 upper=10.0 effort=9.0 velocity=2.208932 -> effort=7.0 velocity=32; type revolute -> continuous
- joint HEBI/shoulder/X5_4: limit lower=-10.0 upper=10.0 effort=9.0 velocity=2.208932 -> effort=7.0 velocity=32; type revolute -> continuous
- joint elbow_end/OUTPUT_JOINT: origin xyz=-0.375 0 0 rpy=3.14157 0 0 -> xyz=0.325 -2.44929359829e-18 0.0 rpy=3.14159265359 0 0
- joint shoulder_bracket/OUTPUT_INTERFACE: origin xyz=0 .04235 .04015 rpy=-1.57075 0 0 -> xyz=0 .0225 .055 rpy=1.57079632679 0 0
- joint shoulder_elbow/OUTPUT_JOINT: origin xyz=-0.38 0 0 rpy=3.14157 0 0 -> xyz=0.33 -2.44929359829e-18 0.0 rpy=3.14159265359 0 0

File: hebiros_description/urdf/x_demo.xacro (robot description, xacro)
@@ -2,11 +2,5 @@
 <robot xmlns:xacro="http://www.ros.org/wiki/xacro" name="arm_demo">
   <!-- *************************** XACRO MACROS *************************** -->
-  <xacro:property name="PI" value="3.1415926535897931" />
-  <!-- load macros for modules -->
-  <xacro:include filename="./x_series_common.xacro"/>
-  <xacro:include filename="./x5.xacro"/>
-  <xacro:include filename="./x_shoulder_bracket.xacro"/>
-  <xacro:include filename="./x_wrist_bracket.xacro"/>
-  <xacro:include filename="./x_tube_link.xacro"/>
+  <xacro:include filename="./x_library.xacro"/>
   <!-- ************************* ROBOT DEFINITION ************************* -->
   <link name="world" />
@@ -19,5 +13,5 @@
   <link name="base">
     <visual>
-      <origin xyz=".125 0 -.0254" rpy="0 0 0" />
+      <origin xyz="-.125 0 -.0254" rpy="0 0 0" />
       <geometry>
         <box size="0.25 0.5 0.0508" />
@@ -26,5 +20,5 @@
     </visual>
     <collision>
-      <origin xyz=".125 0 -.0254" rpy="0 0 0" />
+      <origin xyz="-.125 0 -.0254" rpy="0 0 0" />
       <geometry>
         <box size="0.25 0.5 0.0508" />
@@ -44,9 +38,9 @@
   <!-- joints -->
   <xacro:x5 joint="HEBI/base" child="shoulder_bracket" model="X5_4"/>
-  <xacro:x_wrist_bracket name="shoulder_bracket" child="HEBI/shoulder"/>
+  <xacro:x5_heavy_right_inside_bracket name="shoulder_bracket" child="HEBI/shoulder"/>
   <xacro:x5 joint="HEBI/shoulder" child="shoulder_elbow" model="X5_4"/>
-  <xacro:x_tube_link name="shoulder_elbow" child="HEBI/elbow" length="0.33" twist="0.7"/>
+  <xacro:x_tube_link name="shoulder_elbow" child="HEBI/elbow" extension="0.33" twist="${PI}"/>
   <xacro:x5 joint="HEBI/elbow" child="elbow_end" model="X5_4"/>
-  <xacro:x_tube_link name="elbow_end" child="end_effector" length="0.325" twist="0.6"/>
+  <xacro:x_tube_link name="elbow_end" child="end_effector" extension="0.325" twist="${PI}"/>
   <!-- end link -->
   <link name="end_effector/INPUT_INTERFACE">

File: hebiros_description/urdf/x_tube_link.xacro (robot description, xacro)
@@ -2,59 +2,52 @@
 <robot xmlns:xacro="http://www.ros.org/wiki/xacro">
   <!-- NOTE: joint must match the name of the module -->
-  <xacro:macro name="x_tube_link" params="name child length twist">
+  <xacro:macro name="x_tube_link" params="name child extension twist">
+    <xacro:property name="mass" value="${0.4 * (extension + 0.03) + 0.26}"/>
+    <xacro:property name="edge_to_center" value="${.02}"/>
     <link name="${name}/INPUT_INTERFACE">
       <visual>
-        <origin xyz="-.04 .03 .0075" rpy="0 0 3.14157" />
+        <origin xyz="0 0 0" rpy="0 0 0" />
         <geometry>
-          <mesh filename="package://hebiros_description/meshes/x_output_bracket.stl"/>
+          <mesh filename="package://hebiros_description/meshes/A-2038-02.stl"/>
         </geometry>
         <xacro:black_material/>
       </visual>
       <visual>
-        <origin xyz="${-length/2-.0254} 0 .016075" rpy="0 1.57075 0" />
+        <origin xyz="${extension/2} 0 ${edge_to_center}" rpy="0 1.57075 0" />
         <geometry>
-          <cylinder length="${length-.0254}" radius=".015875" />
+          <cylinder length="${extension-.0254}" radius=".016" />
         </geometry>
         <xacro:silver_material/>
       </visual>
       <visual>
-        <origin xyz="${-length-.0254} -.075 -.0125" rpy="1.57075 0 -1.57075" />
+        <origin xyz="${extension} ${sin(-twist) * edge_to_center} ${edge_to_center * (1 + cos(-twist))}" rpy="${-twist} 0 0"/>
         <geometry>
-          <mesh filename="package://hebiros_description/meshes/x_mounting_bracket.stl"/>
+          <mesh filename="package://hebiros_description/meshes/A-2039-02.stl"/>
         </geometry>
         <xacro:black_material/>
       </visual>
       <collision>
-        <origin xyz="-.04 .03 .0075" rpy="0 0 3.14157" />
+        <origin xyz="0 0 0" rpy="0 0 0" />
         <geometry>
-          <mesh filename="package://hebiros_description/meshes/x_output_bracket.stl"/>
+          <mesh filename="package://hebiros_description/meshes/A-2038-02.stl"/>
         </geometry>
       </collision>
       <collision>
-        <origin xyz="${-length/2-.0254} 0 .016075" rpy="0 1.57075 0" />
+        <origin xyz="${extension/2} 0 ${edge_to_center}" rpy="0 1.57075 0" />
         <geometry>
-          <cylinder length="${length}" radius=".015875" />
+          <cylinder length="${extension-.0254}" radius=".016" />
         </geometry>
       </collision>
       <collision>
-        <origin xyz="${-length-.0254} -.075 -.0125" rpy="1.57075 0 -1.57075" />
+        <origin xyz="${extension} ${sin(-twist) * edge_to_center} ${edge_to_center * (1 + cos(-twist))}" rpy="${-twist} 0 0"/>
         <geometry>
-          <mesh filename="package://hebiros_description/meshes/x_mounting_bracket.stl"/>
+          <mesh filename="package://hebiros_description/meshes/A-2039-02.stl"/>
         </geometry>
       </collision>
+      <!-- Approximate inertia as thin rod about x axis -->
       <inertial>
-        <origin xyz="-.04 .03 .0075" rpy="0 0 3.14157" />
-        <mass value="0.01"/>
-        <inertia  ixx="1.0" ixy="0.0"  ixz="0.0"  iyy="1.0"  iyz="0.0"  izz="1.0"/>
-      </inertial>
-      <inertial>
-        <origin xyz="${-length/2-.0254} 0 .016075" rpy="0 1.57075 0" />
-        <mass value="${length + 0.05}"/>
-        <inertia  ixx="1.0" ixy="0.0"  ixz="0.0"  iyy="1.0"  iyz="0.0"  izz="1.0"/>
-      </inertial>
-      <inertial>
-        <origin xyz="${-length-.0254} -.075 -.0125" rpy="1.57075 0 -1.57075" />
-        <mass value="0.01"/>
-        <inertia  ixx="1.0" ixy="0.0"  ixz="0.0"  iyy="1.0"  iyz="0.0"  izz="1.0"/>
+        <origin xyz="${extension/2} 0 ${edge_to_center}" rpy="0 0 0" />
+        <mass value="${mass}"/>
+        <inertia  ixx="0.0" ixy="0.0"  ixz="0.0"  iyy="${mass * extension * extension / 12.0}"  iyz="0.0"  izz="${mass * extension * extension / 12.0}"/>
       </inertial>
     </link>
@@ -62,5 +55,5 @@
       <parent link="${name}/INPUT_INTERFACE"/>
       <child link="${child}/INPUT_INTERFACE"/>
-      <origin xyz="${-length-.05} 0 0" rpy="3.14157 0 0"/>
+      <origin xyz="${extension} ${-sin(twist) * edge_to_center} ${edge_to_center * (1 + cos(twist))}" rpy="${twist} 0 0"/>
     </joint>
     <gazebo reference="${name}/INPUT_INTERFACE">
