Commit message: Added low pass filter

File: hebiros_description/urdf/x5.xacro (robot description, xacro)
@@ -30,6 +30,6 @@
         <origin xyz="0 0 0.031" rpy="0 0 0"/>
         <axis xyz="0 0 1"/>
-        <limit effort="9.0" lower="-10.0" upper="10.0" velocity="2.208932"/>
-        <dynamics damping="0.5" friction="0.5"/>
+        <limit effort="90.0" lower="-10.0" upper="10.0" velocity="2.208932"/>
+        <dynamics damping="0.2" friction="0.2"/>
       </joint>
     </xacro:if>
@@ -40,6 +40,6 @@
         <origin xyz="0 0 0.031" rpy="0 0 0"/>
         <axis xyz="0 0 1"/>
-        <limit effort="9.0" lower="-10.0" upper="10.0" velocity="2.208932"/>
-        <dynamics damping="0.5" friction="0.5"/>
+        <limit effort="90.0" lower="-10.0" upper="10.0" velocity="2.208932"/>
+        <dynamics damping="0.2" friction="0.2"/>
       </joint>
     </xacro:if>
@@ -50,6 +50,6 @@
         <origin xyz="0 0 0.031" rpy="0 0 0"/>
         <axis xyz="0 0 1"/>
-        <limit effort="9.0" lower="-10.0" upper="10.0" velocity="2.208932"/>
-        <dynamics damping="0.5" friction="0.5"/>
+        <limit effort="90.0" lower="-10.0" upper="10.0" velocity="2.208932"/>
+        <dynamics damping="0.2" friction="0.2"/>
       </joint>
     </xacro:if>

File: hebiros_description/urdf/x_demo.urdf (robot description, URDF)
Before this commit: robot arm_demo, 9 links, 8 joints
Joints:
- removed joint HEBI/base/X5-1
- removed joint HEBI/elbow/X5-9
- added joint HEBI/base/X5-4: type revolute, parent HEBI/base/INPUT_INTERFACE, child shoulder_bracket/INPUT_INTERFACE, origin xyz=0 0 0.031 rpy=0 0 0, axis 0 0 1, limit lower=-10.0 upper=10.0 effort=90.0 velocity=2.208932
- added joint HEBI/elbow/X5-4: type revolute, parent HEBI/elbow/INPUT_INTERFACE, child elbow_end/INPUT_INTERFACE, origin xyz=0 0 0.031 rpy=0 0 0, axis 0 0 1, limit lower=-10.0 upper=10.0 effort=90.0 velocity=2.208932
- joint HEBI/shoulder/X5-4: limit lower=-10.0 upper=10.0 effort=9.0 velocity=2.208932 -> lower=-10.0 upper=10.0 effort=90.0 velocity=2.208932

File: hebiros_description/urdf/x_demo.xacro (robot description, xacro)
@@ -43,9 +43,9 @@
   </joint>
   <!-- joints -->
-  <xacro:x5 joint="HEBI/base" child="shoulder_bracket" model="X5-1"/>
+  <xacro:x5 joint="HEBI/base" child="shoulder_bracket" model="X5-4"/>
   <xacro:x_wrist_bracket name="shoulder_bracket" child="HEBI/shoulder"/>
   <xacro:x5 joint="HEBI/shoulder" child="shoulder_elbow" model="X5-4"/>
   <xacro:x_tube_link name="shoulder_elbow" child="HEBI/elbow" length="0.33" twist="0"/>
-  <xacro:x5 joint="HEBI/elbow" child="elbow_end" model="X5-9"/>
+  <xacro:x5 joint="HEBI/elbow" child="elbow_end" model="X5-4"/>
   <xacro:x_tube_link name="elbow_end" child="end_effector" length="0.325" twist="0"/>
   <!-- end link -->

Commit message: Fix the COM + inertia values for the X5 urdf

File: hebiros_description/urdf/x5.xacro (robot description, xacro)
@@ -19,7 +19,7 @@
       </collision>
       <inertial>
-        <origin xyz="0 0 0.0155" rpy="3.14157 0 0" />
+        <origin xyz="-0.0142, -0.0031, 0.0165" rpy="0 0 0" />
         <mass value="0.335"/>
-        <inertia  ixx="1.0" ixy="0.0"  ixz="0.0"  iyy="1.0"  iyz="0.0"  izz="1.0"/>
+        <inertia ixx="0.00015" iyy="0.000255" izz="0.000350" ixy="0.0000341" ixz="0.0000118" iyz="0.00000229"/>
       </inertial>
     </link>

Commit message: Fixed coordinate system issues with X5 / X8 modules, and updated X tube link definition to add "twist" parameter and fix dimensions, masses and inertias.

File: hebiros_description/urdf/x5.xacro (robot description, xacro)
@@ -6,5 +6,5 @@
     <link name="${joint}/INPUT_INTERFACE">
       <visual>
-        <origin xyz="0 0 0" rpy="0 0 3.1415" />
+        <origin xyz="0 0 0" rpy="0 0 0" />
         <geometry>
           <mesh filename="package://hebiros_description/meshes/x5.stl" scale="0.001 0.001 0.001"/>
@@ -13,5 +13,5 @@
       </visual>
       <collision>
-        <origin xyz="0 0 0" rpy="0 0 3.1415" />
+        <origin xyz="0 0 0" rpy="0 0 0" />
         <geometry>
           <mesh filename="package://hebiros_description/meshes/x5.stl" scale="0.001 0.001 0.001"/>

File: hebiros_description/urdf/x8.xacro (robot description, xacro)
@@ -6,5 +6,5 @@
     <link name="${joint}/INPUT_INTERFACE">
       <visual>
-        <origin xyz="0 0 0" rpy="0 0 3.1415" />
+        <origin xyz="0 0 0" rpy="0 0 0" />
         <geometry>
           <mesh filename="package://hebiros_description/meshes/x8.stl" scale="0.001 0.001 0.001"/>
@@ -13,5 +13,5 @@
       </visual>
       <collision>
-        <origin xyz="0 0 0" rpy="0 0 3.1415" />
+        <origin xyz="0 0 0" rpy="0 0 0" />
         <geometry>
           <mesh filename="package://hebiros_description/meshes/x8.stl" scale="0.001 0.001 0.001"/>

File: hebiros_description/urdf/x_demo.urdf (robot description, URDF)
Before this commit: robot arm_demo, 9 links, 8 joints
Links:
- link elbow_end/INPUT_INTERFACE: mass 0.01 -> 0.402; geometry collision cylinder length=0.2996 radius=.016; collision mesh filename=package://hebiros_description/meshes/PM-2146-02.stl scale=.001 .001 .001
- link shoulder_elbow/INPUT_INTERFACE: mass 0.01 -> 0.404; geometry collision cylinder length=0.3046 radius=.016; collision mesh filename=package://hebiros_description/meshes/PM-2146-02.stl scale=.001 .001 .001
Joints:
- joint elbow_end/OUTPUT_JOINT: origin xyz=-0.375 0 0 rpy=3.14157 0 0 -> xyz=0.325 -0.0189260017537 0.0135342086627 rpy=1.9 0 0
- joint shoulder_elbow/OUTPUT_JOINT: origin xyz=-0.38 0 0 rpy=3.14157 0 0 -> xyz=0.33 -0.00494807918509 0.0393782484342 rpy=0.25 0 0

File: hebiros_description/urdf/x_demo.xacro (robot description, xacro)
@@ -20,5 +20,5 @@
   <link name="base">
     <visual>
-      <origin xyz=".125 0 -.0254" rpy="0 0 0" />
+      <origin xyz="-.125 0 -.0254" rpy="0 0 0" />
       <geometry>
         <box size="0.25 0.5 0.0508" />
@@ -27,5 +27,5 @@
     </visual>
     <collision>
-      <origin xyz=".125 0 -.0254" rpy="0 0 0" />
+      <origin xyz="-.125 0 -.0254" rpy="0 0 0" />
       <geometry>
         <box size="0.25 0.5 0.0508" />
@@ -47,7 +47,7 @@
   <xacro:x_wrist_bracket name="shoulder_bracket" child="HEBI/shoulder"/>
   <xacro:x5 joint="HEBI/shoulder" child="shoulder_elbow" model="X5_4"/>
-  <xacro:x_tube_link name="shoulder_elbow" child="HEBI/elbow" length="0.33" twist="0.7"/>
+  <xacro:x_tube_link name="shoulder_elbow" child="HEBI/elbow" extension="0.33" twist="0.25"/>
   <xacro:x5 joint="HEBI/elbow" child="elbow_end" model="X5_4"/>
-  <xacro:x_tube_link name="elbow_end" child="end_effector" length="0.325" twist="0.6"/>
+  <xacro:x_tube_link name="elbow_end" child="end_effector" extension="0.325" twist="1.9"/>
   <!-- end link -->
   <link name="end_effector/INPUT_INTERFACE">

File: hebiros_description/urdf/x_tube_link.xacro (robot description, xacro)
@@ -2,59 +2,52 @@
 <robot xmlns:xacro="http://www.ros.org/wiki/xacro">
   <!-- NOTE: joint must match the name of the module -->
-  <xacro:macro name="x_tube_link" params="name child length twist">
+  <xacro:macro name="x_tube_link" params="name child extension twist">
+    <xacro:property name="mass" value="${0.4 * (extension + 0.03) + 0.26}"/>
+    <xacro:property name="edge_to_center" value="${.02}"/>
     <link name="${name}/INPUT_INTERFACE">
       <visual>
-        <origin xyz="-.04 .03 .0075" rpy="0 0 3.14157" />
+        <origin xyz="0 0 0" rpy="0 0 0" />
         <geometry>
-          <mesh filename="package://hebiros_description/meshes/x_output_bracket.stl"/>
+          <mesh filename="package://hebiros_description/meshes/PM-2146-02.stl" scale=".001 .001 .001"/>
         </geometry>
         <xacro:black_material/>
       </visual>
       <visual>
-        <origin xyz="${-length/2-.0254} 0 .016075" rpy="0 1.57075 0" />
+        <origin xyz="${extension/2} 0 ${edge_to_center}" rpy="0 1.57075 0" />
         <geometry>
-          <cylinder length="${length-.0254}" radius=".015875" />
+          <cylinder length="${extension-.0254}" radius=".016" />
         </geometry>
         <xacro:silver_material/>
       </visual>
       <visual>
-        <origin xyz="${-length-.0254} -.075 -.0125" rpy="1.57075 0 -1.57075" />
+        <origin xyz="${extension} ${sin(-twist) * edge_to_center} ${edge_to_center * (1 + cos(-twist))}" rpy="${-twist + 3.1415} 0 3.1415"/>
         <geometry>
-          <mesh filename="package://hebiros_description/meshes/x_mounting_bracket.stl"/>
+          <mesh filename="package://hebiros_description/meshes/PM-2147-02.stl" scale=".001 .001 .001"/>
         </geometry>
         <xacro:black_material/>
       </visual>
       <collision>
-        <origin xyz="-.04 .03 .0075" rpy="0 0 3.14157" />
+        <origin xyz="0 0 0" rpy="0 0 0" />
         <geometry>
-          <mesh filename="package://hebiros_description/meshes/x_output_bracket.stl"/>
+          <mesh filename="package://hebiros_description/meshes/PM-2146-02.stl" scale=".001 .001 .001"/>
         </geometry>
       </collision>
       <collision>
-        <origin xyz="${-length/2-.0254} 0 .016075" rpy="0 1.57075 0" />
+        <origin xyz="${extension/2} 0 ${edge_to_center}" rpy="0 1.57075 0" />
         <geometry>
-          <cylinder length="${length}" radius=".015875" />
+          <cylinder length="${extension-.0254}" radius=".016" />
         </geometry>
       </collision>
       <collision>
-        <origin xyz="${-length-.0254} -.075 -.0125" rpy="1.57075 0 -1.57075" />
+        <origin xyz="${extension} ${sin(-twist) * edge_to_center} ${edge_to_center * (1 + cos(-twist))}" rpy="${-twist + 3.1415} 0 3.1415"/>
         <geometry>
-          <mesh filename="package://hebiros_description/meshes/x_mounting_bracket.stl"/>
+          <mesh filename="package://hebiros_description/meshes/PM-2147-02.stl" scale=".001 .001 .001"/>
         </geometry>
       </collision>
+      <!-- Approximate inertia as thin rod about x axis -->
       <inertial>
-        <origin xyz="-.04 .03 .0075" rpy="0 0 3.14157" />
-        <mass value="0.01"/>
-        <inertia  ixx="1.0" ixy="0.0"  ixz="0.0"  iyy="1.0"  iyz="0.0"  izz="1.0"/>
-      </inertial>
-      <inertial>
-        <origin xyz="${-length/2-.0254} 0 .016075" rpy="0 1.57075 0" />
-        <mass value="${length + 0.05}"/>
-        <inertia  ixx="1.0" ixy="0.0"  ixz="0.0"  iyy="1.0"  iyz="0.0"  izz="1.0"/>
-      </inertial>
-      <inertial>
-        <origin xyz="${-length-.0254} -.075 -.0125" rpy="1.57075 0 -1.57075" />
-        <mass value="0.01"/>
-        <inertia  ixx="1.0" ixy="0.0"  ixz="0.0"  iyy="1.0"  iyz="0.0"  izz="1.0"/>
+        <origin xyz="${extension/2} 0 ${edge_to_center}" rpy="0 0 0" />
+        <mass value="${mass}"/>
+        <inertia  ixx="0.0" ixy="0.0"  ixz="0.0"  iyy="${mass * extension * extension / 12.0}"  iyz="0.0"  izz="${mass * extension * extension / 12.0}"/>
       </inertial>
     </link>
@@ -62,5 +55,5 @@
       <parent link="${name}/INPUT_INTERFACE"/>
       <child link="${child}/INPUT_INTERFACE"/>
-      <origin xyz="${-length-.05} 0 0" rpy="3.14157 0 0"/>
+      <origin xyz="${extension} ${-sin(twist) * edge_to_center} ${edge_to_center * (1 + cos(twist))}" rpy="${twist} 0 0"/>
     </joint>
     <gazebo reference="${name}/INPUT_INTERFACE">

Commit message: Plugin in progress

File: hebiros_description/urdf/x5.xacro (robot description, xacro)
@@ -19,5 +19,5 @@
       </collision>
       <inertial>
-        <origin xyz="-0.0142, -0.0031, 0.0165" rpy="0 0 0" />
+        <origin xyz="-0.0142 -0.0031 0.0165" rpy="0 0 0" />
         <mass value="0.335"/>
         <inertia ixx="0.00015" iyy="0.000255" izz="0.000350" ixy="0.0000341" ixz="0.0000118" iyz="0.00000229"/>

Commit message: Restructure tested and functional

File: hebiros_description/urdf/x5.xacro (robot description, xacro)
@@ -31,5 +31,8 @@
         <axis xyz="0 0 1"/>
         <limit effort="9.0" lower="-10.0" upper="10.0" velocity="2.208932"/>
-        <dynamics damping="0.5" friction="0.5"/>
+        <dynamics damping="0.1" friction="0.1"/>
+        <physics>
+          <provide_feedback>true</provide_feedback>
+        </physics>
       </joint>
     </xacro:if>
@@ -41,5 +44,5 @@
         <axis xyz="0 0 1"/>
         <limit effort="9.0" lower="-10.0" upper="10.0" velocity="2.208932"/>
-        <dynamics damping="0.5" friction="0.5"/>
+        <dynamics damping="0.1" friction="0.1"/>
       </joint>
     </xacro:if>
@@ -51,17 +54,7 @@
         <axis xyz="0 0 1"/>
         <limit effort="9.0" lower="-10.0" upper="10.0" velocity="2.208932"/>
-        <dynamics damping="0.5" friction="0.5"/>
+        <dynamics damping="0.1" friction="0.1"/>
       </joint>
     </xacro:if>
-    <transmission name="${joint}/transmission">
-    <type>transmission_interface/SimpleTransmission</type>
-      <joint name="${joint}">
-        <hardwareInterface>hardware_interface/EffortJointInterface</hardwareInterface>
-      </joint>
-      <actuator name="${joint}/actuator">
-        <hardwareInterface>hardware_interface/EffortJointInterface</hardwareInterface>
-        <mechanicalReduction>1</mechanicalReduction>
-      </actuator>
-    </transmission>
     <gazebo reference="${joint}/INPUT_INTERFACE">
       <selfCollide>true</selfCollide>

Commit message: Created urdfs for various kits

File: hebiros_description/urdf/x5.xacro (robot description, xacro)
@@ -80,4 +80,5 @@
         <pose>0 0 0 0 0 0</pose>
       </sensor>
+      <material>Gazebo/BlueGlow</material>
     </gazebo>
   </xacro:macro>

File: hebiros_description/urdf/x_tube_link.xacro (robot description, xacro)
@@ -59,4 +59,5 @@
     <gazebo reference="${name}/INPUT_INTERFACE">
       <selfCollide>true</selfCollide>
+      <material>Gazebo/FlatBlack</material>
     </gazebo>
   </xacro:macro>
