Commit message: STL files

File: hebiros_description/urdf/rosie.xacro (robot description, xacro)
@@ -63,5 +63,5 @@
       <origin xyz="0 0 0" rpy="0 0 0"/>
       <geometry>
-        <mesh filename="package://turtlebot3_description/meshes/sensors/lds.stl" scale="0.001 0.001 0.001"/>
+        <mesh filename="package://hebiros_description/meshes/lds.stl" scale="0.001 0.001 0.001"/>
       </geometry>
       <material name="dark"/>

Commit message: Ipad Controller Integration

File: hebiros_description/urdf/rosie.xacro (robot description, xacro)
@@ -57,5 +57,5 @@
     <parent link="base_link"/>
     <child link="base_scan"/>
-    <origin xyz="-0.064 0 0.122" rpy="0 0 0"/>
+    <origin xyz="-0.064 0 0.122" rpy="0 0 1.5708"/>
   </joint>
   <link name="base_scan">

Commit message: updated parameters

File: hebiros_description/urdf/rosie.xacro (robot description, xacro)
@@ -13,5 +13,5 @@
       <origin xyz="-0 0 0" rpy="0 0 0"/>
       <geometry>
-        <box size="0.30 0.30 0.10"/>
+        <box size="0.50 0.50 0.10"/>
         <mesh filename="package://hebiros_description/meshes/A-2127-02_Simple.stl" scale="0.001 0.001 0.001"/>
       </geometry>
@@ -21,5 +21,5 @@
       <origin xyz="0 0 0" rpy="0 0 0"/>
       <geometry>
-        <box size="0.3 0.3 0.1"/>
+        <box size="0.50 0.50 0.1"/>
       </geometry>
     </collision>

Commit message: posting latest code

File: hebiros_description/urdf/rosie.xacro (robot description, xacro)
@@ -11,8 +11,8 @@
   <link name="base_link">
     <visual>
-      <origin xyz="-0 0 0" rpy="0 0 0"/>
+      <origin xyz="-0.1625 0.1775 0" rpy="1.5708 0 0"/>
       <geometry>
-        <box size="0.50 0.50 0.10"/>
-        <mesh filename="package://hebiros_description/meshes/A-2127-02_Simple.stl" scale="0.001 0.001 0.001"/>
+        <!--box size="0.50 0.50 0.10"/-->
+        <mesh filename="package://hebiros_description/meshes/rosie_simplified_1.stl" scale="0.001 0.001 0.001"/>
       </geometry>
       <material name="light_black"/>
@@ -25,9 +25,9 @@
     </collision>
   </link>
-<!--
+<!---->
   <joint name="Wheel1_joint" type="fixed">
     <parent link="base_link"/>
     <child link="HEBI/Wheel1/INPUT_INTERFACE"/>
-    <origin xyz="0.0 0.15 0.0" rpy="0 1.5708 1.5708"/>
+    <origin xyz="0.0680 0.135 0.030" rpy="0.523599 1.5708 1.5708"/>
     <axis xyz="0 0 1"/>
   </joint>
@@ -35,5 +35,5 @@
     <parent link="base_link"/>
     <child link="HEBI/Wheel2/INPUT_INTERFACE"/>
-    <origin xyz="0.0 -0.15 0.0" rpy="0 1.5708 -1.5708"/>
+    <origin xyz="0.0680 -0.135 0.030" rpy="-0.523599 1.5708 -1.5708"/>
     <axis xyz="0 0 1"/>
   </joint>
@@ -41,5 +41,5 @@
     <parent link="base_link"/>
     <child link="HEBI/Wheel3/INPUT_INTERFACE"/>
-    <origin xyz="-0.15 0.0 0.0" rpy="0 1.5708 3.14159"/>
+    <origin xyz="-0.155 0.0 0.030" rpy="0 1.5708 3.14159"/>
     <axis xyz="0 0 1"/>
   </joint>
@@ -48,14 +48,35 @@
   <xacro:x5 joint="HEBI/Wheel3" child="omniwheel3" model="X5_4"/>
   <link name="omniwheel1/INPUT_INTERFACE">
+    <visual>
+      <origin xyz="0.1030 0.185 0.050" rpy="0.523599 1.5708 1.5708"/>
+      <geometry>
+        <!--box size="0.50 0.50 0.10"/-->
+        <mesh filename="package://hebiros_description/meshes/omni_25k.stl" scale="0.001 0.001 0.001"/>
+      </geometry>
+    </visual>
   </link>
   <link name="omniwheel2/INPUT_INTERFACE">
+    <visual>
+      <origin xyz="0.0930 -0.175 0.050" rpy="-0.523599 1.5708 1.5708"/>
+      <geometry>
+        <!--box size="0.50 0.50 0.10"/-->
+        <mesh filename="package://hebiros_description/meshes/omni_25k.stl" scale="0.001 0.001 0.001"/>
+      </geometry>
+    </visual>
   </link>
   <link name="omniwheel3/INPUT_INTERFACE">
+    <visual>
+      <origin xyz="-0.220 0 0.050" rpy="0 1.5708 3.14159"/>
+      <geometry>
+        <!--box size="0.50 0.50 0.10"/-->
+        <mesh filename="package://hebiros_description/meshes/omni_25k.stl" scale="0.001 0.001 0.001"/>
+      </geometry>
+    </visual>
   </link>
-  -->
+  <!-- -->
   <joint name="scan_joint" type="fixed">
     <parent link="base_link"/>
     <child link="base_scan"/>
-    <origin xyz="-0.064 0 0.122" rpy="0 0 1.5708"/>
+    <origin xyz="0 0 0.180" rpy="0 0 1.5708"/>
   </joint>
   <link name="base_scan">
