Commit message: XACRO updates

File: hebiros_description/urdf/omnibase.xacro (robot description, xacro)
@@ -97,5 +97,5 @@
       <origin xyz="0 0 0.030" rpy="0 0 0"/>
       <geometry>
-        <mesh filename="package://hebiros_description/meshes/omni_25k.stl" scale="0.001 0.001 0.001"/>
+        <mesh filename="package://hebiros_description/meshes/omniwheels.stl" scale="0.001 0.001 0.001"/>
       </geometry>
       <material name="light_black"/>
@@ -106,5 +106,5 @@
       <origin xyz="0 0 0.030" rpy="0 0 0"/>
       <geometry>
-        <mesh filename="package://hebiros_description/meshes/omni_25k.stl" scale="0.001 0.001 0.001"/>
+        <mesh filename="package://hebiros_description/meshes/omniwheels.stl" scale="0.001 0.001 0.001"/>
       </geometry>
       <material name="light_black"/>
@@ -115,5 +115,5 @@
       <origin xyz="0 0 .030 " rpy="0 0 0"/>
       <geometry>
-        <mesh filename="package://hebiros_description/meshes/omni_25k.stl" scale="0.001 0.001 0.001"/>
+        <mesh filename="package://hebiros_description/meshes/omniwheels.stl" scale="0.001 0.001 0.001"/>
       </geometry>
       <material name="light_black"/>

Commit message: Review fixes

File: hebiros_description/urdf/omnibase.xacro (robot description, xacro)
@@ -1,5 +1,4 @@
 <?xml version="1.0" ?>
 <robot name="rosie_test" xmlns:xacro="http://www.ros.org/wiki/xacro">
-  <xacro:include filename="$(find hebiros_description)/urdf/common_properties.xacro"/>
   <xacro:include filename="$(find hebiros_description)/urdf/x_library.xacro"/>
   <xacro:include filename="$(find hebiros_description)/urdf/x_series_common.xacro"/>
@@ -29,5 +28,5 @@
   <joint name="module1_joint" type="fixed">
     <parent link="base_link"/>
-    <child link="HEBI/Module1"/>
+    <child link="module1"/>
     <origin xyz="0.055 0.110 0.030" rpy="0.523599 1.5708 1.5708"/>
     <axis xyz="0 0 1"/>
@@ -35,5 +34,5 @@
   <joint name="module2_joint" type="fixed">
     <parent link="base_link"/>
-    <child link="HEBI/Module2"/>
+    <child link="module2"/>
     <origin xyz="0.055 -0.110 0.030" rpy="-0.523599 1.5708 -1.5708"/>
     <axis xyz="0 0 1"/>
@@ -41,9 +40,9 @@
   <joint name="module3_joint" type="fixed">
     <parent link="base_link"/>
-    <child link="HEBI/Module3"/>
+    <child link="module3"/>
     <origin xyz="-0.125 0.0 0.030" rpy="0 1.5708 3.14159"/>
     <axis xyz="0 0 1"/>
   </joint>
-  <link name="HEBI/Module1">
+  <link name="module1">
     <visual>
       <origin xyz="0 0 0.030" rpy="0 0 0"/>
@@ -55,5 +54,5 @@
     </visual>
   </link>
-  <link name="HEBI/Module2">
+  <link name="module2">
     <visual>
       <origin xyz="0 0 0.030" rpy="0 0 0"/>
@@ -65,5 +64,5 @@
     </visual>
   </link>
-  <link name="HEBI/Module3">
+  <link name="module3">
     <visual>
       <origin xyz="0 0 .030 " rpy="0 0 0"/>
@@ -76,5 +75,5 @@
   </link>
   <joint name="omniwheel1_joint" type="fixed">
-    <parent link="HEBI/Module1"/>
+    <parent link="module1"/>
     <child link="omniwheel1"/>
     <origin xyz="0 0 .060" rpy="0 0 0"/>
@@ -82,5 +81,5 @@
   </joint>
   <joint name="omniwheel2_joint" type="fixed">
-    <parent link="HEBI/Module2"/>
+    <parent link="module2"/>
     <child link="omniwheel2"/>
     <origin xyz="0 0 0.060" rpy="0 0 0"/>
@@ -88,5 +87,5 @@
   </joint>
   <joint name="omniwheel3_joint" type="fixed">
-    <parent link="HEBI/Module3"/>
+    <parent link="module3"/>
     <child link="omniwheel3"/>
     <origin xyz="0.0 0.0 0.060" rpy="0 0 0"/>
@@ -120,5 +119,5 @@
     </visual>
   </link>
-  <!-- LIDAR Information-->
+  <!-- LIDAR Module Information-->
   <joint name="scan_joint" type="fixed">
     <parent link="base_link"/>
@@ -130,8 +129,15 @@
       <origin xyz="0 0 0" rpy="0 0 0"/>
       <geometry>
-        <mesh filename="package://hebiros_description/meshes/lds.stl" scale="0.001 0.001 0.001"/>
+        <mesh filename="package://hebiros_description/meshes/simple_lidar.stl" scale="0.001 0.001 0.001"/>
       </geometry>
       <material name="dark"/>
     </visual>
   </link>
+  <!-- Color Parameters-->
+  <material name="dark">
+    <color rgba="0.3 0.3 0.3 1.0"/>
+  </material>
+  <material name="light_black">
+    <color rgba="0.4 0.4 0.4 1.0"/>
+  </material>
 </robot>
